File: Eagle files/Jar_of_Fireflies.sch (EAGLE design)
At the start: 14 parts, among them IC1 ATTINY85

Commit message: Overdue updates
Parts:
- removed JP1, JP2: STAND-OFF, SparkFun:STAND-OFF
- added R4: (no value), resistor:R-US_0204/7
- LED1, LED2, LED3, LED4, LED5, LED6: device SparkFun:LED3MM -> SparkFun:LED5MM
- R1, R3: device resistor:R-US_0204/5 -> resistor:R-US_0207/2V
- R2: device resistor:R-US_0204/5 -> resistor:R-US_0204/7
Connections:
- net 1+ renamed PORTA
- net 2+ renamed PORTB
- removed net 1-: IC1.PB2(SCK/ADC1), LED1.C, LED4.C
- removed net 2-: IC1.PB3(ADC3), LED2.C, LED5.C
- removed net 3-: IC1.PB5(NRES), LED3.C, LED6.C
- new net N$3: LED3.A, LED4.C, LED5.A, LED6.C, R3.2
- new net PORTC: IC1.PB2(SCK/ADC1), R3.1
- net GND: now also R4.1; no longer R3.1
- net N$1: now also LED2.C, LED3.C, LED4.A, R2.2; no longer LED2.A, LED3.A, R1.2
- net N$2: now also LED1.C, LED2.A, LED5.C, R1.2; no longer LED4.A, LED5.A, R2.2
- net PIEZO: now also R4.2; no longer R3.2
- net VCC: now also IC1.PB5(NRES)
Other:
- note added: "Charlieplexed LEDs"
- note added: "Microcontroller"
- note added: "Piezo element"
- note added: "Power in"
- note removed: "LEDs"
- note removed: "MICROCONTROLLER"
- note removed: "PIEZO"
- note removed: "POWER"
- moved on the sheet: IC1, LED1, LED2, LED3, LED4, LED5, LED6, PIEZO, POWER, R1, R2, R3
